File: JukePCB/Jukebox/Jukebox.sch (EAGLE design)
At the start: 31 parts, among them CN1 1X4-BIG

Commit message: Huge Sound Update, almost final
Parts:
- added A3, A4: 1k, SparkFun-Resistors:10KOHM-HORIZ-1/4W-1%
Connections:
- new net N$38: A3.1, A4.1, TOLIGHT.TIP
- net GND: now also TOLIGHT.RING
- net N$23: now also A3.2; no longer TOLIGHT.RING
- net N$24: now also A4.2; no longer TOLIGHT.TIP
Changed lines of the file:
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@@
 <part name="CONTROL1" library="adafruit" deviceset="1X4" device="-BIG"/>
 <part name="CONTROL2" library="adafruit" deviceset="1X4" device="-BIG"/>
+<part name="A3" library="SparkFun-Resistors" deviceset="10KOHM" device="-HORIZ-1/4W-1%" value="1k"/>
+<part name="A4" library="SparkFun-Resistors" deviceset="10KOHM" device="-HORIZ-1/4W-1%" value="1k"/>
 </parts>
 <sheets>
@@
 <instance part="CONTROL1" gate="G$1" x="-33.02" y="7.62" rot="R180"/>
 <instance part="CONTROL2" gate="G$1" x="-33.02" y="-5.08" rot="R180"/>
+<instance part="A3" gate="G$1" x="213.36" y="12.7"/>
+<instance part="A4" gate="G$1" x="213.36" y="17.78"/>
 </instances>
 <busses>
@@
 <pinref part="AUXOUT" gate="G$1" pin="RING"/>
 <wire x1="198.12" y1="25.4" x2="246.38" y2="25.4" width="0.1524" layer="91"/>
-<pinref part="TOLIGHT" gate="G$1" pin="RING"/>
-<wire x1="198.12" y1="12.7" x2="246.38" y2="12.7" width="0.1524" layer="91"/>
 <wire x1="246.38" y1="12.7" x2="246.38" y2="25.4" width="0.1524" layer="91"/>
 <junction x="246.38" y="25.4"/>
+<pinref part="A3" gate="G$1" pin="2"/>
+<wire x1="218.44" y1="12.7" x2="246.38" y2="12.7" width="0.1524" layer="91"/>
 </segment>
 </net>
@@
 <pinref part="AUXOUT" gate="G$1" pin="TIP"/>
 <wire x1="198.12" y1="30.48" x2="251.46" y2="30.48" width="0.1524" layer="91"/>
-<pinref part="TOLIGHT" gate="G$1" pin="TIP"/>
-<wire x1="198.12" y1="17.78" x2="251.46" y2="17.78" width="0.1524" layer="91"/>
 <wire x1="251.46" y1="17.78" x2="251.46" y2="30.48" width="0.1524" layer="91"/>
 <junction x="251.46" y="30.48"/>
+<pinref part="A4" gate="G$1" pin="2"/>
+<wire x1="251.46" y1="17.78" x2="218.44" y2="17.78" width="0.1524" layer="91"/>
 </segment>
 </net>
@@
 <pinref part="TOLIGHT" gate="G$1" pin="GND"/>
 <wire x1="187.96" y1="15.24" x2="182.88" y2="15.24" width="0.1524" layer="91"/>
-<wire x1="182.88" y1="15.24" x2="182.88" y2="0" width="0.1524" layer="91"/>
+<wire x1="182.88" y1="15.24" x2="182.88" y2="2.54" width="0.1524" layer="91"/>
 <junction x="182.88" y="15.24"/>
+<wire x1="182.88" y1="2.54" x2="182.88" y2="0" width="0.1524" layer="91"/>
 <wire x1="182.88" y1="15.24" x2="182.88" y2="27.94" width="0.1524" layer="91"/>
 <junction x="182.88" y="27.94"/>
@@
 <wire x1="182.88" y1="58.42" x2="182.88" y2="71.12" width="0.1524" layer="91"/>
 <wire x1="182.88" y1="71.12" x2="187.96" y2="71.12" width="0.1524" layer="91"/>
+<pinref part="TOLIGHT" gate="G$1" pin="RING"/>
+<wire x1="198.12" y1="12.7" x2="198.12" y2="2.54" width="0.1524" layer="91"/>
+<wire x1="198.12" y1="2.54" x2="182.88" y2="2.54" width="0.1524" layer="91"/>
+<junction x="182.88" y="2.54"/>
 </segment>
 <segment>
@@
 </segment>
 </net>
+<net name="N$38" class="0">
+<segment>
+<pinref part="TOLIGHT" gate="G$1" pin="TIP"/>
+<pinref part="A4" gate="G$1" pin="1"/>
+<wire x1="208.28" y1="17.78" x2="203.2" y2="17.78" width="0.1524" layer="91"/>
+<pinref part="A3" gate="G$1" pin="1"/>
+<wire x1="203.2" y1="17.78" x2="198.12" y2="17.78" width="0.1524" layer="91"/>
+<wire x1="208.28" y1="12.7" x2="203.2" y2="12.7" width="0.1524" layer="91"/>
+<wire x1="203.2" y1="12.7" x2="203.2" y2="17.78" width="0.1524" layer="91"/>
+<junction x="203.2" y="17.78"/>
+</segment>
+</net>
