File: JukePCB/Jukebox/Jukebox.brd (EAGLE design)
At the start: 133.5 x 197 mm, 33 parts, among them CN1 1X4-BIG

Commit message: Probably final board
Parts:
- moved A4 0.50 mm to (-41.0, 8.50)
Routing:
- net N$27: track 214.7 -> 217.1 mm
- net N$22: track 116.4 -> 118.3 mm
- net N$37: track 126.8 -> 128.7 mm
- net N$34: track 117.3 -> 119.2 mm
- net N$25: track 117.9 -> 119.8 mm
- net N$23: track 27.7 -> 29.3 mm
- net N$24: track 46.1 -> 46.6 mm
Changed lines of the file:
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@@
 <attribute name="PROD_ID" value="RES-12183" x="-25" y="8" size="1.778" layer="27" display="off"/>
 </element>
-<element name="A4" library="SparkFun-Resistors" package="AXIAL-0.3" value="1k" x="-41" y="9" rot="R90">
-<attribute name="PROD_ID" value="RES-12183" x="-41" y="9" size="1.778" layer="27" rot="R90" display="off"/>
+<element name="A4" library="SparkFun-Resistors" package="AXIAL-0.3" value="1k" x="-41" y="8.5" rot="R90">
+<attribute name="PROD_ID" value="RES-12183" x="-41" y="8.5" size="1.778" layer="27" rot="R90" display="off"/>
 </element>
 </elements>
@@
 <contactref element="A3" pad="P$2"/>
 <wire x1="-20.06" y1="20.75" x2="-20.06" y2="21.25" width="0.4064" layer="16"/>
-<wire x1="-21.19" y1="8" x2="-21.19" y2="13.12" width="0.4064" layer="16"/>
 <wire x1="-34.5" y1="23.5" x2="-22.81" y2="23.5" width="0.4064" layer="16"/>
 <wire x1="-22.81" y1="23.5" x2="-20.06" y2="20.75" width="0.4064" layer="16"/>
-<wire x1="-20.06" y1="14.25" x2="-21.19" y2="13.12" width="0" layer="19" extent="16-16"/>
+<wire x1="-21.19" y1="8" x2="-21.19" y2="13.12" width="0.4064" layer="16"/>
+<wire x1="-21.19" y1="13.12" x2="-20.06" y2="14.25" width="0.4064" layer="16"/>
 </signal>
 <signal name="N$24">
@@
 <wire x1="-34.5" y1="28.5" x2="-20.31" y2="28.5" width="0.4064" layer="16"/>
 <wire x1="-20.31" y1="28.5" x2="-20.06" y2="28.25" width="0.4064" layer="16"/>
-<wire x1="-41" y1="12.81" x2="-41" y2="26.5" width="0.4064" layer="16"/>
 <wire x1="-41" y1="26.5" x2="-39" y2="28.5" width="0.4064" layer="16"/>
 <wire x1="-39" y1="28.5" x2="-34.5" y2="28.5" width="0.4064" layer="16"/>
+<wire x1="-41" y1="26.5" x2="-41" y2="12.31" width="0.4064" layer="16"/>
 </signal>
 <signal name="N$27">
@@
 <wire x1="66" y1="57" x2="66" y2="21" width="0.4064" layer="16"/>
 <wire x1="66" y1="21" x2="60" y2="15" width="0.4064" layer="16"/>
-<wire x1="60" y1="15" x2="54" y2="15" width="0.4064" layer="16"/>
-<wire x1="54" y1="15" x2="28.57" y2="15" width="0.4064" layer="16"/>
+<wire x1="60" y1="15" x2="28.57" y2="15" width="0.4064" layer="16"/>
 <wire x1="28.57" y1="15" x2="14.84" y2="28.73" width="0.4064" layer="16"/>
 <wire x1="60.25" y1="-58.25" x2="60.25" y2="-41.25" width="0.4064" layer="16"/>
-<wire x1="60.25" y1="-41.25" x2="54" y2="-35" width="0.4064" layer="16"/>
-<wire x1="54" y1="-35" x2="54" y2="15" width="0.4064" layer="16"/>
+<wire x1="60.25" y1="-41.25" x2="54.125" y2="-35.125" width="0.4064" layer="16"/>
 <wire x1="13.81" y1="-16" x2="13.81" y2="0.24" width="0.4064" layer="16"/>
 <wire x1="13.81" y1="0.24" x2="28.57" y2="15" width="0.4064" layer="1"/>
 <via x="13.81" y="0.24" extent="1-16" drill="0.6" shape="square"/>
 <via x="28.57" y="15" extent="1-16" drill="0.6" shape="square"/>
+<wire x1="60" y1="15" x2="54" y2="9" width="0.4064" layer="16"/>
+<wire x1="54" y1="9" x2="54" y2="-35" width="0.4064" layer="16"/>
+<wire x1="54" y1="-35" x2="54.125" y2="-35.125" width="0.4064" layer="16"/>
 </signal>
 <signal name="N$8">
@@
 <wire x1="36.69" y1="33.81" x2="49.5" y2="21" width="0.4064" layer="16"/>
 <wire x1="49.5" y1="21" x2="49.5" y2="-55.5" width="0.4064" layer="1"/>
-<wire x1="49.5" y1="-55.5" x2="60.25" y2="-66.25" width="0.4064" layer="16"/>
 <via x="49.5" y="21" extent="1-16" drill="0.6" shape="square"/>
 <via x="49.5" y="-55.5" extent="1-16" drill="0.6" shape="square"/>
+<wire x1="60.25" y1="-66.25" x2="57" y2="-66.25" width="0.4064" layer="16"/>
+<wire x1="57" y1="-66.25" x2="49.5" y2="-58.75" width="0.4064" layer="16"/>
+<wire x1="49.5" y1="-58.75" x2="49.5" y2="-55.5" width="0.4064" layer="16"/>
 </signal>
 <signal name="N$25">
@@
 <wire x1="36.73" y1="31.27" x2="47" y2="21" width="0.4064" layer="16"/>
 <wire x1="47" y1="21" x2="47" y2="-57" width="0.4064" layer="1"/>
-<wire x1="47" y1="-57" x2="60.25" y2="-70.25" width="0.4064" layer="16"/>
 <via x="47" y="21" extent="1-16" drill="0.6" shape="square"/>
 <via x="47" y="-57" extent="1-16" drill="0.6" shape="square"/>
+<wire x1="60.25" y1="-70.25" x2="57" y2="-70.25" width="0.4064" layer="16"/>
+<wire x1="57" y1="-70.25" x2="47" y2="-60.25" width="0.4064" layer="16"/>
+<wire x1="47" y1="-60.25" x2="47" y2="-57" width="0.4064" layer="16"/>
 </signal>
 <signal name="N$34">
@@
 <wire x1="41.85" y1="23.65" x2="44.5" y2="21" width="0.4064" layer="16"/>
 <wire x1="44.5" y1="21" x2="44.5" y2="-58.5" width="0.4064" layer="1"/>
-<wire x1="44.5" y1="-58.5" x2="60.25" y2="-74.25" width="0.4064" layer="16"/>
 <via x="44.5" y="21" extent="1-16" drill="0.6" shape="square"/>
 <via x="44.5" y="-58.5" extent="1-16" drill="0.6" shape="square"/>
+<wire x1="60.25" y1="-74.25" x2="57" y2="-74.25" width="0.4064" layer="16"/>
+<wire x1="57" y1="-74.25" x2="44.5" y2="-61.75" width="0.4064" layer="16"/>
+<wire x1="44.5" y1="-61.75" x2="44.5" y2="-58.5" width="0.4064" layer="16"/>
 </signal>
 <signal name="N$37">
@@
 <via x="42" y="21" extent="1-16" drill="0.6" shape="square"/>
 <via x="42" y="-68" extent="1-16" drill="0.6" shape="square"/>
-<wire x1="42" y1="-68" x2="60.25" y2="-86.25" width="0.4064" layer="16"/>
+<wire x1="60.25" y1="-86.25" x2="57" y2="-86.25" width="0.4064" layer="16"/>
+<wire x1="57" y1="-86.25" x2="42" y2="-71.25" width="0.4064" layer="16"/>
+<wire x1="42" y1="-71.25" x2="42" y2="-68" width="0.4064" layer="16"/>
 </signal>
 <signal name="N$13">
@@
 <wire x1="-28.5" y1="40.75" x2="-28.5" y2="32.75" width="0.4064" layer="16"/>
 <wire x1="-28.5" y1="32.75" x2="-29" y2="32.25" width="0.4064" layer="16"/>
-<wire x1="-29" y1="32.25" x2="-40.5" y2="32.25" width="0.4064" layer="16"/>
-<wire x1="-40.5" y1="32.25" x2="-46.75" y2="26" width="0.4064" layer="16"/>
-<wire x1="-46.75" y1="26" x2="-46.75" y2="12.75" width="0.4064" layer="16"/>
-<wire x1="-46.75" y1="12.75" x2="-41" y2="7" width="0.4064" layer="16"/>
+<wire x1="-29" y1="32.25" x2="-40.75" y2="32.25" width="0.4064" layer="16"/>
+<wire x1="-46.5" y1="12.5" x2="-41" y2="7" width="0.4064" layer="16"/>
 <wire x1="-41" y1="7" x2="-35.5" y2="7" width="0.4064" layer="16"/>
 <wire x1="-35.5" y1="7" x2="-31" y2="11.5" width="0.4064" layer="16"/>
 <wire x1="-31" y1="11.5" x2="-31" y2="13" width="0.4064" layer="16"/>
 <wire x1="-31" y1="13" x2="-34.5" y2="16.5" width="0.4064" layer="16"/>
+<wire x1="-40.75" y1="32.25" x2="-46.5" y2="26.5" width="0.4064" layer="16"/>
+<wire x1="-46.5" y1="26.5" x2="-46.5" y2="12.5" width="0.4064" layer="16"/>
 </signal>
 <signal name="N$14">
@@
 <wire x1="-26" y1="32.75" x2="-28" y2="30.75" width="0.4064" layer="16"/>
 <wire x1="-28" y1="30.75" x2="-39.5" y2="30.75" width="0.4064" layer="16"/>
-<wire x1="-39.5" y1="30.75" x2="-44.25" y2="26" width="0.4064" layer="16"/>
-<wire x1="-44.25" y1="26" x2="-44.25" y2="12.75" width="0.4064" layer="16"/>
-<wire x1="-44.25" y1="12.75" x2="-41" y2="9.5" width="0.4064" layer="16"/>
 <wire x1="-41" y1="9.5" x2="-36.5" y2="9.5" width="0.4064" layer="16"/>
 <wire x1="-36.5" y1="9.5" x2="-34.5" y2="11.5" width="0.4064" layer="16"/>
+<wire x1="-39.5" y1="30.75" x2="-43.75" y2="26.5" width="0.4064" layer="16"/>
+<wire x1="-43.75" y1="26.5" x2="-43.75" y2="12.25" width="0.4064" layer="16"/>
+<wire x1="-43.75" y1="12.25" x2="-41" y2="9.5" width="0.4064" layer="16"/>
 </signal>
 <signal name="N$15">
@@
 <contactref element="TOLIGHT" pad="2"/>
 <contactref element="A4" pad="P$1"/>
-<wire x1="-41" y1="5.19" x2="-35.19" y2="5.19" width="0.4064" layer="16"/>
-<wire x1="-35.19" y1="5.19" x2="-34.5" y2="4.5" width="0.4064" layer="16"/>
 <contactref element="A3" pad="P$1"/>
 <wire x1="-28.81" y1="8" x2="-31" y2="8" width="0.4064" layer="16"/>
 <wire x1="-31" y1="8" x2="-34.5" y2="4.5" width="0.4064" layer="16"/>
+<wire x1="-41" y1="4.69" x2="-34.5" y2="4.69" width="0.4064" layer="16"/>
+<wire x1="-34.5" y1="4.69" x2="-34.5" y2="4.5" width="0.4064" layer="16"/>
 </signal>
 </signals>
